Commit message: 4

File: src/dog/description/robot_core.xacro (robot description, xacro)
@@ -28,19 +28,108 @@
     <link name="chassis">
         <visual>
-            <origin xyz="0.055 0 0.04"/>
-            <geometry>
-                <box size="0.11 0.09 0.08"/>
+            <origin xyz="0.055 0 0.0015"/>
+            <geometry>
+                <box size="0.11 0.09 0.03"/>
             </geometry>
             <material name="blue"/>
         </visual>
         <collision>
-            <origin xyz="0.055 0 0.04"/>
-            <geometry>
-                <box size="0.11 0.09 0.08"/>
-            </geometry>
-        </collision>
-        <xacro:inertial_box mass="0.5" x="0.11" y="0.09" z="0.08">
-            <origin xyz="0.055 0 0.04" rpy="0 0 0"/>
+            <origin xyz="0.055 0 0.0015"/>
+            <geometry>
+                <box size="0.11 0.09 0.03"/>
+            </geometry>
+        </collision>
+        <xacro:inertial_box mass="0.5" x="0.11" y="0.09" z="0.03">
+            <origin xyz="0.055 0 0.0015" rpy="0 0 0"/>
         </xacro:inertial_box>
+    </link>
+                <!-- PILLAR -->
+    <joint name="pillar_1_joint" type="fixed">
+        <parent link="chassis"/>
+        <child link="pillar_1_link"/>
+        <origin xyz="0.015 0 0.03"/>
+    </joint>
+    <link name="pillar_1_link">
+        <visual>
+            <origin xyz="0 0.035 0"/>
+            <geometry>
+                <cylinder radius="0.0035" length="0.03"/>
+            </geometry>
+            <material name="orange"/>
+        </visual>
+        <collision>
+            <geometry>
+                <cylinder radius="0.0035" length="0.03"/>
+            </geometry>
+        </collision>
+        <xacro:inertial_cylinder mass="0.01" length="0.03" radius="0.0035">
+            <origin xyz="0 0 0" rpy="0 0 0"/>
+        </xacro:inertial_cylinder>
+    </link>
+    <joint name="pillar_2_joint" type="fixed">
+        <parent link="chassis"/>
+        <child link="pillar_2_link"/>
+        <origin xyz="0.015 0 0.03"/>
+    </joint>
+    <link name="pillar_2_link">
+        <visual>
+            <origin xyz="0 -0.035 0"/>
+            <geometry>
+                <cylinder radius="0.0035" length="0.03"/>
+            </geometry>
+            <material name="orange"/>
+        </visual>
+        <collision>
+            <geometry>
+                <cylinder radius="0.0035" length="0.03"/>
+            </geometry>
+        </collision>
+        <xacro:inertial_cylinder mass="0.5" length="0.03" radius="0.0035">
+            <origin xyz="0 0 0" rpy="0 0 0"/>
+        </xacro:inertial_cylinder>
+    </link>
+    <joint name="pillar_3_joint" type="fixed">
+        <parent link="chassis"/>
+        <child link="pillar_3_link"/>
+        <origin xyz="0.095 0 0.03"/>
+    </joint>
+    <link name="pillar_3_link">
+        <visual>
+            <origin xyz="0 -0.035 0"/>
+            <geometry>
+                <cylinder radius="0.0035" length="0.03"/>
+            </geometry>
+            <material name="orange"/>
+        </visual>
+        <collision>
+            <geometry>
+                <cylinder radius="0.0035" length="0.03"/>
+            </geometry>
+        </collision>
+        <xacro:inertial_cylinder mass="0.5" length="0.03" radius="0.0035">
+            <origin xyz="0 0 0" rpy="0 0 0"/>
+        </xacro:inertial_cylinder>
+    </link>
+    <joint name="pillar_4_joint" type="fixed">
+        <parent link="chassis"/>
+        <child link="pillar_4_link"/>
+        <origin xyz="0.095 0 0.03"/>
+    </joint>
+    <link name="pillar_4_link">
+        <visual>
+            <origin xyz="0 0.035 0"/>
+            <geometry>
+                <cylinder radius="0.0035" length="0.03"/>
+            </geometry>
+            <material name="orange"/>
+        </visual>
+        <collision>
+            <geometry>
+                <cylinder radius="0.0035" length="0.03"/>
+            </geometry>
+        </collision>
+        <xacro:inertial_cylinder mass="0.01" length="0.03" radius="0.0035">
+            <origin xyz="0 0 0" rpy="0 0 0"/>
+        </xacro:inertial_cylinder>
     </link>
     <!-- LEFT WHEEL LINK -->

File: src/dog/description/robot_lidar.xacro (robot description, xacro)
@@ -8,7 +8,7 @@
     <link name="lidar_link">
         <visual>
-            <origin xyz="0.001 0 0" rpy="0 0 0"/>
+            <origin xyz="0.0005 0 0" rpy="0 0 0"/>
             <geometry>
-                <box size="0.0001 0.03 0.01"/>
+                <box size="0.001 0.055 0.023"/>
             </geometry>
             <material name="black"/>
@@ -16,5 +16,5 @@
         <collision>
             <geometry>
-                <box size="0.0001 0.03 0.01"/>
+                <box size="0.001 0.055 0.023"/>
             </geometry>
         </collision>
@@ -23,5 +23,5 @@
         <parent link="lidar_link"/>
         <child link="T_link"/>
-        <origin xyz="0.015 0 0" rpy="0 0 0"/>
+        <origin xyz="0 0.015 0" rpy="0 0 0"/>
     </joint>
     <link name="T_link">
@@ -42,5 +42,5 @@
         <parent link="lidar_link"/>
         <child link="R_link"/>
-        <origin xyz="-0.015 0 0" rpy="${pi/2} 0 ${pi/2}"/>
+        <origin xyz="0 -0.015 0" rpy="${pi/2} 0 ${pi/2}"/>
     </joint>
     <link name="R_link">
