Commit message: 123

File: src/dog/description/robot.urdf.xacro (robot description, xacro)
@@ -2,4 +2,6 @@
 <robot xmlns:xacro="http://www.ros.org/wiki/xacro"  name="robot">
     <xacro:include filename="robot_core.xacro" />
-    <xacro:include filename="robot_lidar.xacro"/>
+    <!-- <xacro:include filename="robot_gazebo.xacro"/> -->
+    <xacro:include filename="ros2_control.xacro"/>
+    <!-- <xacro:include filename="robot_lidar.xacro"/> -->
 </robot>

File: src/dog/description/robot_core.xacro (robot description, xacro)
@@ -28,5 +28,5 @@
     <link name="chassis">
         <visual>
-            <origin xyz="0.055 0 0.0015"/>
+            <origin xyz="0.055 0 0.015"/>
             <geometry>
                 <box size="0.11 0.09 0.03"/>
@@ -35,102 +35,16 @@
         </visual>
         <collision>
-            <origin xyz="0.055 0 0.0015"/>
+            <origin xyz="0.055 0 0.015"/>
             <geometry>
                 <box size="0.11 0.09 0.03"/>
             </geometry>
         </collision>
-        <xacro:inertial_box mass="0.5" x="0.11" y="0.09" z="0.03">
-            <origin xyz="0.055 0 0.0015" rpy="0 0 0"/>
+        <xacro:inertial_box mass="0.05" x="0.11" y="0.09" z="0.03">
+            <origin xyz="0.055 0 0.015" rpy="0 0 0"/>
         </xacro:inertial_box>
     </link>
-                <!-- PILLAR -->
-    <joint name="pillar_1_joint" type="fixed">
-        <parent link="chassis"/>
-        <child link="pillar_1_link"/>
-        <origin xyz="0.015 0 0.03"/>
-    </joint>
-    <link name="pillar_1_link">
-        <visual>
-            <origin xyz="0 0.035 0"/>
-            <geometry>
-                <cylinder radius="0.0035" length="0.03"/>
-            </geometry>
-            <material name="orange"/>
-        </visual>
-        <collision>
-            <geometry>
-                <cylinder radius="0.0035" length="0.03"/>
-            </geometry>
-        </collision>
-        <xacro:inertial_cylinder mass="0.01" length="0.03" radius="0.0035">
-            <origin xyz="0 0 0" rpy="0 0 0"/>
-        </xacro:inertial_cylinder>
-    </link>
-    <joint name="pillar_2_joint" type="fixed">
-        <parent link="chassis"/>
-        <child link="pillar_2_link"/>
-        <origin xyz="0.015 0 0.03"/>
-    </joint>
-    <link name="pillar_2_link">
-        <visual>
-            <origin xyz="0 -0.035 0"/>
-            <geometry>
-                <cylinder radius="0.0035" length="0.03"/>
-            </geometry>
-            <material name="orange"/>
-        </visual>
-        <collision>
-            <geometry>
-                <cylinder radius="0.0035" length="0.03"/>
-            </geometry>
-        </collision>
-        <xacro:inertial_cylinder mass="0.5" length="0.03" radius="0.0035">
-            <origin xyz="0 0 0" rpy="0 0 0"/>
-        </xacro:inertial_cylinder>
-    </link>
-    <joint name="pillar_3_joint" type="fixed">
-        <parent link="chassis"/>
-        <child link="pillar_3_link"/>
-        <origin xyz="0.095 0 0.03"/>
-    </joint>
-    <link name="pillar_3_link">
-        <visual>
-            <origin xyz="0 -0.035 0"/>
-            <geometry>
-                <cylinder radius="0.0035" length="0.03"/>
-            </geometry>
-            <material name="orange"/>
-        </visual>
-        <collision>
-            <geometry>
-                <cylinder radius="0.0035" length="0.03"/>
-            </geometry>
-        </collision>
-        <xacro:inertial_cylinder mass="0.5" length="0.03" radius="0.0035">
-            <origin xyz="0 0 0" rpy="0 0 0"/>
-        </xacro:inertial_cylinder>
-    </link>
-    <joint name="pillar_4_joint" type="fixed">
-        <parent link="chassis"/>
-        <child link="pillar_4_link"/>
-        <origin xyz="0.095 0 0.03"/>
-    </joint>
-    <link name="pillar_4_link">
-        <visual>
-            <origin xyz="0 0.035 0"/>
-            <geometry>
-                <cylinder radius="0.0035" length="0.03"/>
-            </geometry>
-            <material name="orange"/>
-        </visual>
-        <collision>
-            <geometry>
-                <cylinder radius="0.0035" length="0.03"/>
-            </geometry>
-        </collision>
-        <xacro:inertial_cylinder mass="0.01" length="0.03" radius="0.0035">
-            <origin xyz="0 0 0" rpy="0 0 0"/>
-        </xacro:inertial_cylinder>
-    </link>
+    <gazebo reference="chassis">
+        <material>Gazebo/Blue</material>
+    </gazebo>
     <!-- LEFT WHEEL LINK -->
     <joint name="left_wheel_joint" type="continuous">
@@ -152,8 +66,11 @@
             </geometry>
         </collision>
-        <xacro:inertial_cylinder mass="0.1" length="0.03" radius="0.015">
+        <xacro:inertial_cylinder mass="0.05" length="0.03" radius="0.015">
             <origin xyz="0 0 0" rpy="0 0 0"/>
         </xacro:inertial_cylinder>
     </link>
+    <gazebo reference="left_wheel">
+        <material>Gazebo/Black</material>
+    </gazebo>
     <!-- RIGHT WHEEL LINK -->
     <joint name="right_wheel_joint" type="continuous">
@@ -175,8 +92,11 @@
             </geometry>
         </collision>
-        <xacro:inertial_cylinder mass="0.1" length="0.03" radius="0.0015">
+        <xacro:inertial_cylinder mass="0.05" length="0.03" radius="0.0015">
             <origin xyz="0 0 0" rpy="0 0 0"/>
         </xacro:inertial_cylinder>
     </link>
+    <gazebo reference="right_wheel">
+        <material>Gazebo/Black</material>
+    </gazebo>
     <!-- CASTER WHEEL LINK -->
     <joint name="caster_wheel_joint" type="fixed">
@@ -188,5 +108,5 @@
         <visual>
             <geometry>
-                <sphere radius="0.01"/>
+                <sphere radius="0.02"/>
             </geometry>
             <material name="black"/>
@@ -194,10 +114,15 @@
         <collision>
             <geometry>
-                <sphere radius="0.01"/>
+                <sphere radius="0.03"/>
             </geometry>
         </collision>
-        <xacro:inertial_sphere mass="0.1" radius="0.05">
+        <xacro:inertial_sphere mass="0.02" radius="0.02">
             <origin xyz="0 0 0" rpy="0 0 0"/>
         </xacro:inertial_sphere>
     </link>
+    <gazebo reference="caster_wheel">
+        <material>Gazebo/Black</material>
+        <mu1 value="0.001"/>
+        <mu2 value="0.001"/>
+    </gazebo>
 </robot>

File: src/dog/description/robot_lidar.xacro (robot description, xacro)
@@ -1,3 +1,3 @@
-<?xml version="1.0"?>
+<!-- <?xml version="1.0"?>
 <robot xmlns:xacro="http://www.ros.org/wiki/xacro"  name="robot">
     <joint name="lidar_joint" type="fixed">
@@ -58,3 +58,3 @@
         </collision>
     </link>
-</robot>
+</robot> -->
